Commit message: add HAP and mid360 dae 3D model and 120 degree * 25 degree Vehical-grade lidar simulation model

File: scout_gazebo/urdf/base.xacro (robot description, xacro)
@@ -45,6 +45,6 @@
         <origin rpy="0 0 0" xyz="0 0 0.3" />
     </xacro:realsense_d435> -->
+    <xacro:include filename="$(find scout_gazebo)/urdf/laser_support.xacro" />
     <!-- VLP16 激光雷达 -->
-    <xacro:include filename="$(find scout_gazebo)/urdf/laser_support.xacro" />
     <!-- <xacro:include filename="$(find velodyne_description)/urdf/VLP-16.urdf.xacro"/>
     <xacro:VLP-16 parent="support" name="velodyne" topic="/scan" organize_cloud="${organize_cloud}"
@@ -52,6 +52,15 @@
           <origin xyz="0 0 ${support_length/2}" rpy="0 0 0" />
     </xacro:VLP-16> -->
-    <xacro:include filename="$(find livox_laser_simulation)/urdf/livox_avia.xacro" />
-    <xacro:Livox_Mid40 name="livox" parent="support" />
+    <!-- 车载120°激光雷达 -->
+    <xacro:include filename="$(find velodyne_description)/urdf/Lidar.urdf.xacro" />
+    <xacro:Lidar parent="support" name="lidar" topic="/scan" hz="10"
+        organize_cloud="${organize_cloud}" gpu="${gpu}"
+        samples="480" min_horizonal_angle="-${60.0*M_PI/180.0}" max_horizonal_angle="${60.0*M_PI/180.0}"
+        lasers="96" min_vertical_angle="-${12.5*M_PI/180.0}" max_vertical_angle="${12.5*M_PI/180.0}">
+        <origin xyz="0 0 0.0" rpy="0 0 0" />
+    </xacro:Lidar>
+    <!-- Livox Avia激光雷达 -->
+    <!-- <xacro:include filename="$(find livox_laser_simulation)/urdf/livox_avia.xacro" />
+    <xacro:Livox_AVIA name="livox" parent="support" /> -->
     <!-- IMU 模块 -->
     <xacro:include filename="$(find scout_gazebo)/urdf/imu.xacro" />

File: velodyne_simulator/velodyne_description/urdf/HDL-32E.urdf.xacro (robot description, xacro)
@@ -45,4 +45,9 @@
         </geometry>
       </visual>
+      <collision>
+        <geometry>
+          <sphere radius="0"/>
+        </geometry>
+      </collision>
     </link>
     <!-- Gazebo requires the velodyne_gazebo_plugins package -->

File: velodyne_simulator/velodyne_description/urdf/VLP-16.urdf.xacro (robot description, xacro)
@@ -50,4 +50,9 @@
         </geometry>
       </visual>
+      <collision>
+        <geometry>
+          <sphere radius="0"/>
+        </geometry>
+      </collision>
     </link>
     <!-- Gazebo requires the velodyne_gazebo_plugins package -->
@@ -81,5 +86,5 @@
               <type>gaussian</type>
               <mean>0.0</mean>
-              <stddev>0.01</stddev>
+              <stddev>0.0</stddev>
             </noise>
           </ray>

File: velodyne_simulator/velodyne_description/urdf/example.urdf.xacro (robot description, xacro)
@@ -40,3 +40,9 @@
     <origin xyz="0 0 0.6" rpy="0 0 0" />
   </xacro:HDL-32E>
+  <!-- <xacro:include filename="$(find velodyne_description)/urdf/Lidar.urdf.xacro"/>
+  <xacro:Lidar parent="base_link" name="lidar" topic="/scan" hz="10" organize_cloud="${organize_cloud}" gpu="${gpu}"
+  samples="480" min_horizonal_angle="-${60.0*M_PI/180.0}" max_horizonal_angle="${60.0*M_PI/180.0}"
+  lasers="96" min_vertical_angle="-${12.5*M_PI/180.0}" max_vertical_angle="${12.5*M_PI/180.0}">
+    <origin xyz="0 0 0.2" rpy="0 0 0" />
+  </xacro:Lidar> -->
 </robot>
